File: power_module_v2test.kicad_pcb (KiCad board)
At the start: 4 copper layers, 95 x 66 mm, 71 parts, among them J1 USB_C_PD, J2 OUTPUT, J3 I2C_BREAKOUT, Q1 DUAL_N_FET, Q2 DUAL_N_FET, Q3 DUAL_N_FET, Q4 DUAL_N_FET, SW1 ON_OFF, U1 BQ7692003, U2 CH224K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

Commit message: more changes
Parts:
- moved C16 54.1 mm to (32.9, 23.0)
- moved R12 51.0 mm to (33.7, 31.3)
- moved C10 49.7 mm to (33.8, 24.9)
- moved U3 47.5 mm to (37.9, 22.9)
- moved R11 46.9 mm to (36.5, 26.8)
- moved C12 46.3 mm to (38.7, 19.4)
- moved C14 43.2 mm to (39.6, 25.9)
- moved R13 41.5 mm to (41.6, 24.2)
- moved R14 41.4 mm to (38.2, 29.7)
- moved Q2 39.8 mm to (43.2, 12.4)
- moved L1 38.5 mm to (53.3, 15.6)
- moved C13 37.4 mm to (42.1, 19.9)
- moved R26 28.7 mm to (89.6, 52.6)
- moved C21 28.5 mm to (92.6, 51.8)
- moved R10 28.5 mm to (55.4, 25.5)
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