File: power_module.kicad_pcb (KiCad board)
At the start: 4 copper layers, 95 x 66 mm, 71 parts, among them J1 USB_C_PD, J2 OUTPUT, J3 I2C_BREAKOUT, Q1 DUAL_N_FET, Q2 DUAL_N_FET, Q3 DUAL_N_FET, Q4 DUAL_N_FET, SW1 ON_OFF, U1 BQ7692003, U2 CH224K, U3 BQ24650, U4 LM5176PWPR

Commit message: PCB: add 4 BAT1 stitch vias on west-side cell terminals
Bridges BAT1's B.Cu pads to the In1.Cu tracks freerouting left
floating. Closes 4 of 10 BAT1 unconnects: BAT1.1 BAT+, BAT1.3
CELL2_TOP, BAT1.5 CELL1_TOP, BAT1.6 BAT-.

East-side BAT1 vias (BAT1.2 CELL2_TOP, BAT1.4 CELL1_TOP) attempted
but rolled back — the 0.6 mm vias short into nearby freerouting
F.Cu traces at the BAT1 east-edge area. Hand-fix needed: either
move those tracks or use a smaller via and offset the via slightly
from pad center.

State: 50 errors / 16 unconnected remaining.

Co-Authored-By: Claude Opus 4.7 <noreply@anthropic.com>
Routing:
- net CELL2_TOP: vias 3 -> 4
- net CELL1_TOP: vias 3 -> 4
- net BAT-: vias 2 -> 3
- net BAT+: vias 7 -> 8
Changed lines of the file:
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@@
 	)
 	(via
+		(at 4.854 49.448)
+		(size 0.6)
+		(drill 0.3)
+		(layers "F.Cu" "B.Cu")
+		(net 1)
+	)
+	(via
 		(at 77.7804 51.4039)
 		(size 1)
@@
 	)
 	(via
+		(at 87.154 12.448)
+		(size 0.6)
+		(drill 0.3)
+		(layers "F.Cu" "B.Cu")
+		(net 31)
+	)
+	(via
 		(at 17.2009 24.0125)
 		(size 1)
@@
 	)
 	(via
+		(at 4.854 30.948)
+		(size 0.6)
+		(drill 0.3)
+		(layers "F.Cu" "B.Cu")
+		(net 50)
+	)
+	(via
 		(at 39.9231 35.9332)
 		(size 0.6)
@@
 		(net 55)
 	)
+	(via
+		(at 4.854 12.448)
+		(size 0.6)
+		(drill 0.3)
+		(layers "F.Cu" "B.Cu")
+		(net 55)
+	)
