File: power_module.kicad_pcb (KiCad board)
At the start: 4 copper layers, 95 x 76.9 mm, 71 parts, among them J1 USB_C_PD, J2 OUTPUT, J3 I2C_BREAKOUT, Q1 DUAL_N_FET, Q2 DUAL_N_FET, Q3 DUAL_N_FET, Q4 DUAL_N_FET, SW1 ON_OFF, U1 BQ7692003, U2 CH224K, U3 BQ24650, U4 LM5176PWPR

Commit message: Working on fixing unconnects etc
Parts:
- moved C22 12.4 mm to (58.9, 70.4), turned to 180 degrees
- moved C29 7.59 mm to (58.4, 73.7), turned to -90 degrees
- moved R22 1.24 mm to (73.9, 62.7), turned to 90 degrees
- moved C8 0.75 mm to (70.9, 62.9)
- moved Q4 0.61 mm to (62.7, 58.9)
- turned R24 to 180 degrees
Routing:
- net BAT+: track 74.8 -> 115.4 mm, vias 13 -> 17
- net V12_OUT: track 94.8 -> 59.5 mm, vias 3 -> 2
- net BB_SW2: track 51.9 -> 32.5 mm
- net BB_EN: track 44.6 -> 28.1 mm
- net CELL1_TOP: track 85.6 -> 100.8 mm, vias 0 -> 2
- net V12_INT: track 38.6 -> 27.8 mm
- net GND: track 105.8 -> 116.3 mm, vias 34 -> 36
- net BB_BOOT1: track 34.3 -> 24.7 mm
- net BB_SLOPE: track 26.8 -> 23.4 mm
- net CELL2_TOP: track 84.4 -> 87.6 mm, vias 0 -> 1
- net BB_FB: track 39.3 -> 37.0 mm
- net BB_SS: track 0.00 -> 2.23 mm
- net BAT-: track 141.8 -> 143.8 mm, vias 1 -> 2
- net BB_RT: track 21.3 -> 22.7 mm
