File: bms.kicad_sch (KiCad schematic)
At the start: 22 parts, among them Q1 DUAL_N_FET, U1 BQ7692003

Commit message: Moved U4 to bottom, away from pads and away from cells.  Swapped SMD thermistor for THT and moved to B.Cu.  Locked thermistor and BAT1.
Parts:
- BAT1: now not fitted
- TH1: value NTC_10k -> 103AT NTC 10k +-3%; footprint Resistor_SMD:R_0603_1608Metric -> Resistor_THT:R_Axial_DIN0204_L3.6mm_D1.6mm_P1.90mm_Vertical; LCSC C13564 -> (none); now not fitted
