File: bms.kicad_sch (KiCad schematic)
At the start: 22 parts, among them Q1 DUAL_N_FET, U1 BQ7692003

Commit message: annotate bypass caps with Pin_Spring_Class:1 = DECOUPLING
C3, C4 (bms.kicad_sch) and C29, C30 (buckboost.kicad_sch) are
bypass / decoupling caps that need to sit right next to their IC
pin during placement. With this annotation the auto-placer
(relax_placement) parks them at <1 mm from the target IC pin
instead of leaving them at the default 5+ mm.

Reads at session-load time per #228, so no PCB-side sync needed.

Co-Authored-By: Claude Opus 4.7 <noreply@anthropic.com>
Parts:
- C3, C4: Pin_Spring_Class:1 (none) -> DECOUPLING
Changed lines of the file:
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@@
 			)
 		)
+    (property "Pin_Spring_Class:1" "DECOUPLING" (at 195.0 70.0 0)
+      (effects (font (size 1.27 1.27)) (hide yes))
+    )
 		(pin "2"
 		)
@@
 			)
 		)
-		(pin "2"
-		)
+    (property "Pin_Spring_Class:1" "DECOUPLING" (at 195.0 55.0 0)
+      (effects (font (size 1.27 1.27)) (hide yes))
+    )
+		(pin "2"
+		)
