File: buckboost.kicad_sch (KiCad schematic)
At the start: 25 parts, among them Q3 DUAL_N_FET, Q4 DUAL_N_FET, U4 LM5176

Commit message: Moved U4 to bottom, away from pads and away from cells.  Swapped SMD thermistor for THT and moved to B.Cu.  Locked thermistor and BAT1.
Connections:
- net BB_SW1: no longer C23.2, U4.16 (CS)
- new net: C23.2, U4.16 (CS)
