File: charger.kicad_sch (KiCad schematic)
At the start: 21 parts, among them J1 USB_C_PD, Q2 DUAL_N_FET, U2 CH224K, U3 BQ24650

Commit message: charger: per-target spring annotations + selective autoplace of U3 group
Annotate U3's decoupling/bulk/bootstrap caps with per-target
Pin_Spring_Class ({"U3.N": "DECOUPLING"}) so each is pulled onto the
specific pin it serves rather than everything on its rail; status LED
D1 weakly tethered (INTER_GROUP). Classify USB_VBUS as INTER_GROUP in
the META1 spring-class net map (cross-group rail; stops Q2 drifting to
the input side). Selectively relax the charger satellites with U3
anchored and all other groups locked.

Co-Authored-By: Claude Opus 4.7 <noreply@anthropic.com>
Parts:
- C10, C16: Pin_Spring_Class:1 (none) -> {"U3.1": "DECOUPLING"}
- C12: Pin_Spring_Class:1 (none) -> {"U3.16": "DECOUPLING"}
- C13: Pin_Spring_Class:1 (none) -> {"U3.12": "DECOUPLING"}
- C14: Pin_Spring_Class:1 (none) -> {"U3.6": "DECOUPLING"}
- C15: Pin_Spring_Class:1 (none) -> {"U3.9": "DECOUPLING"}
- D1: Pin_Spring_Class:1 (none) -> {"U3.3": "INTER_GROUP"}
Changed lines of the file:
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@@
 			)
 		)
+    (property "Pin_Spring_Class:1" "{\"U3.1\": \"DECOUPLING\"}" (at 255.0 88.0 0)
+      (effects (font (size 1.27 1.27)) (hide yes))
+    )
 		(pin "1"
 		)
@@
 			)
 		)
+    (property "Pin_Spring_Class:1" "{\"U3.16\": \"DECOUPLING\"}" (at 285.0 95.0 0)
+      (effects (font (size 1.27 1.27)) (hide yes))
+    )
 		(pin "1"
 		)
@@
 			)
 		)
+    (property "Pin_Spring_Class:1" "{\"U3.1\": \"DECOUPLING\"}" (at 240.0 88.0 0)
+      (effects (font (size 1.27 1.27)) (hide yes))
+    )
 		(pin "2"
 		)
@@
 			)
 		)
+    (property "Pin_Spring_Class:1" "{\"U3.3\": \"INTER_GROUP\"}" (at 305.0 80.0 0)
+      (effects (font (size 1.27 1.27)) (hide yes))
+    )
 		(pin "2"
 		)
@@
 			)
 		)
+    (property "Pin_Spring_Class:1" "{\"U3.12\": \"DECOUPLING\"}" (at 285.0 100.0 0)
+      (effects (font (size 1.27 1.27)) (hide yes))
+    )
 		(pin "2"
 		)
@@
 			)
 		)
+    (property "Pin_Spring_Class:1" "{\"U3.6\": \"DECOUPLING\"}" (at 290.0 105.0 0)
+      (effects (font (size 1.27 1.27)) (hide yes))
+    )
 		(pin "2"
 		)
@@
 			)
 		)
-		(pin "2"
-		)
+    (property "Pin_Spring_Class:1" "{\"U3.9\": \"DECOUPLING\"}" (at 295.0 115.0 0)
+      (effects (font (size 1.27 1.27)) (hide yes))
+    )
+		(pin "2"
+		)
