File: power_module.kicad_sch (KiCad schematic)
At the start: 4 parts, among them J2 OUTPUT, J3 I2C_BREAKOUT, SW1 ON_OFF

Commit message: charger: incremental autoroute of 6/8 BQ signal nets
First use of the new incremental autoroute (MCP #242): routed
BQ_PH/BQ_VREF/BQ_VFB/BQ_BTST/BQ_LODRV/CHG_OUT (+69 tracks, +5 vias),
leaving all non-charger copper byte-identical. refill_zones run after.

Hand-off state for review: BQ_HIDRV and BQ_STAT1 still open, and ~8
clashes remain where the freshly-routed charger tracks meet the existing
USB_VBUS pour / fixed pads (the incremental-route caveat — freerouting
optimized against a re-routed scratch layout). DRC 108 total.

(.kicad_sch: verify_netclass_patterns bootstrapped the
mcp_expected_netclass_patterns metadata property — purely additive.)
Parts:
- META1: mcp_expected_netclass_patterns (none) -> [{"netclass":"POWER_4A","pattern":"BAT+"},{"netclass":"POWE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
Changed lines of the file:
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@@
+			)
+		)
+		(property "mcp_expected_netclass_patterns" "[{\"netclass\":\"POWER_4A\",\"pattern\":\"BAT+\"},{\"netclass\":\"POWER_4A\",\"pattern\":\"BAT-\"},{\"netclass\":\"POWER_4A\",\"pattern\":\"V12_OUT\"},{\"netclass\":\"POWER_2A\",\"pattern\":\"USB_VBUS\"},{\"netclass\":\"POWER_2A\",\"pattern\":\"CHG_OUT\"},{\"netclass\":\"POWER_2A\",\"pattern\":\"BQ_PH\"}]"
+			(at 12.7 12.7 0)
+			(effects
+				(font
+					(size 1.27 1.27)
+				)
+				(hide yes)
 			)
 		)
